File: linear_encoder.kicad_pcb (KiCad board)
At the start: 2 copper layers, 35 x 33 mm, 8 parts, among them J1 Conn_01x08, U1 TXB0104PW

Commit message: Layout & Schematic
Parts:
- added C1: 100n, Capacitor_SMD:C_0805_2012Metric, F.Cu at (87.5, 30.5)
- added C2: 100n, Capacitor_SMD:C_0805_2012Metric, F.Cu at (97.0, 30.5)
Routing:
- net +5V: track 21.7 -> 2.80 mm
- net GND: track 16.2 -> 22.7 mm, vias 0 -> 1
- net +3V3: track 28.9 -> 33.5 mm
